File: hardware/cn910-breakout-kicad/cn910-breakout.kicad_pcb (KiCad board)
At the start: 2 copper layers, 62.7 x 64.5 mm, 51 parts, among them J1 CN910, J2 USB4125-GF-A-0190_REVA2, J3 PB_RF_OUT, J4 RF_AGC_IN, J5 RF_AGC_OUT, J6 CAP_FG, J7 RF_SWP, Q101 NPN, Q111 NPN, Q121 NMOS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

Commit message: Refined routing
Other:
- board text added: "JLCJLCJLCJLC"
Changed lines of the file:
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@@
+		)
+	)
+	(gr_text "JLCJLCJLCJLC"
+		(at 115.45 117.3 0)
+		(layer "B.SilkS")
+		(effects
+			(font
+				(size 1 1)
+				(thickness 0.15)
+			)
+			(justify mirror)
 		)
 	)

Commit message: Refactored CN910 breakout KiCad project files, updating footprint and symbol references to "GDH" naming convention. Adjusted PCB thickness and dielectric properties for improved design accuracy. Added new adhesive layers and updated project metadata with a new variant description. Removed obsolete libraries and 3D models to streamline the project.
Parts:
- G***: footprint GDH_Technologies:gdh_wordmark -> GDH Graphics:gdh_wordmark
- J1: footprint CN910 Breakout Footprints:CON_527461671_MOL -> GDH Connectors:CON_527461671_MOL
- J2: footprint CN910 Breakout Footprints:GCT_USB4125-GF-A-0190_REVA2 -> GDH Connectors:GCT_USB4125-GF-A-0190_REVA2
- J3: footprint CN910 Breakout Footprints:Molex_0731000154_BNC_RA_THT -> GDH Connectors:Molex_0731000154_BNC_RA_THT
- J4, J5, J6, J7: footprint CN910 Breakout Footprints:GRADCONN_RFPC-SMA28-F -> GDH Connectors:GRADCONN_RFPC-SMA28-F
- SW1: footprint CN910 Breakout Footprints:Slide_Switch_SS12D07_CNK -> GDH Switches:Slide_Switch_SS12D07_CNK
Changed lines of the file:
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@@
 	(generator_version "10.0")
 	(general
-		(thickness 1.57)
+		(thickness 1.6)
 		(legacy_teardrops no)
 	)
@@
 		(0 "F.Cu" signal)
 		(2 "B.Cu" signal)
+		(9 "F.Adhes" user "F.Adhesive")
+		(11 "B.Adhes" user "B.Adhesive")
 		(13 "F.Paste" user)
 		(15 "B.Paste" user)
@@
 		(17 "Dwgs.User" user "User.Drawings")
 		(19 "Cmts.User" user "User.Comments")
+		(21 "Eco1.User" user "User.Eco1")
+		(23 "Eco2.User" user "User.Eco2")
 		(25 "Edge.Cuts" user)
 		(27 "Margin" user)
@@
 		(35 "F.Fab" user)
 		(33 "B.Fab" user)
+		(39 "User.1" user)
+		(41 "User.2" user)
+		(43 "User.3" user)
+		(45 "User.4" user)
 	)
 	(setup
@@
 			(layer "dielectric 1"
 				(type "core")
-				(thickness 1.48)
+				(thickness 1.51)
 				(material "FR4")
-				(epsilon_r 4.4)
+				(epsilon_r 4.5)
 				(loss_tangent 0.02)
 			)
@@
 		(capping no)
 		(filling no)
+		(zone_defaults)
 		(pcbplotparams
 			(layerselection 0x00000000_00000000_55555555_5755f5ff)
@@
 		(embedded_fonts no)
 	)
-	(footprint "GDH_Technologies:gdh_wordmark"
+	(footprint "GDH Graphics:gdh_wordmark"
 		(layer "F.Cu")
 		(at 110.551598 56.983015)
@@
 		)
 	)
-	(footprint "CN910 Breakout Footprints:CON_527461671_MOL"
+	(footprint "GDH Connectors:CON_527461671_MOL"
 		(layer "F.Cu")
 		(at 91.9 74.7 -90)
@@
 		)
 	)
-	(footprint "CN910 Breakout Footprints:GRADCONN_RFPC-SMA28-F"
+	(footprint "GDH Connectors:GRADCONN_RFPC-SMA28-F"
 		(layer "F.Cu")
 		(at 110.25 112.19 90)
@@
 		)
 	)
-	(footprint "CN910 Breakout Footprints:GRADCONN_RFPC-SMA28-F"
+	(footprint "GDH Connectors:GRADCONN_RFPC-SMA28-F"
 		(layer "F.Cu")
 		(at 101.25 112.19 180)
@@
 		)
 	)
-	(footprint "CN910 Breakout Footprints:GRADCONN_RFPC-SMA28-F"
+	(footprint "GDH Connectors:GRADCONN_RFPC-SMA28-F"
 		(layer "F.Cu")
 		(at 129.24 112.2 180)
@@
 		)
 	)
-	(footprint "CN910 Breakout Footprints:GRADCONN_RFPC-SMA28-F"
+	(footprint "GDH Connectors:GRADCONN_RFPC-SMA28-F"
 		(layer "F.Cu")
 		(at 120.2 112.2)
@@
 		)
 	)
-	(footprint "CN910 Breakout Footprints:Slide_Switch_SS12D07_CNK"
+	(footprint "GDH Switches:Slide_Switch_SS12D07_CNK"
 		(layer "F.Cu")
 		(at 101.45 63.5 -90)
@@
 		)
 	)
-	(footprint "CN910 Breakout Footprints:GCT_USB4125-GF-A-0190_REVA2"
+	(footprint "GDH Connectors:GCT_USB4125-GF-A-0190_REVA2"
 		(layer "F.Cu")
 		(at 146.2 110.6 90)
@@
 		)
 	)
-	(footprint "CN910 Breakout Footprints:Molex_0731000154_BNC_RA_THT"
+	(footprint "GDH Connectors:Molex_0731000154_BNC_RA_THT"
 		(layer "F.Cu")
 		(at 120.9 73.6 -90)

Commit message: Updated CN910 breakout KiCad project files with dynamic project metadata, including title, company, version, and license. Refined design rules and component properties for improved clarity and organization. Adjusted pin functions and descriptions for connectors, and removed obsolete library references. Enhanced layout with new wire connections and updated schematic components.
Connections:
- net /CN910 Breakout + Raspberry Pi Pico/LANC Interface/LANC_TX_OD renamed /Pi Pico/LANC Interface/LANC_TX_OD
- net /CN910 Breakout + Raspberry Pi Pico/PICO_LANC1_RX_N renamed /Pi Pico/PICO_LANC1_RX_N
- net /CN910 Breakout + Raspberry Pi Pico/PICO_LANC2_RX_N renamed /Pi Pico/PICO_LANC2_RX_N
- net /CN910 Breakout + Raspberry Pi Pico/PICO_LANC_TX renamed /Pi Pico/PICO_LANC_TX
Routing:
- net GND: track 6.07 -> 9.03 mm
