File: kicad-cn910/full/cn910-breakout.kicad_sch (KiCad schematic)
At the start: 30 parts, among them J1 CN910, J2 USB4125-GF-A-0190_REVA2, J3 PB_RF_OUT, SW1 SW_SPDT, U1 ADA4857-1YRZ

Commit message: Refactor code structure for improved readability and maintainability
Parts:
- removed C4: 10u, Capacitor_SMD:C_0603_1608Metric_Pad1.08x0.95mm_HandSolder, symbol Device:C
- removed C5: 100n, Capacitor_SMD:C_0603_1608Metric_Pad1.08x0.95mm_HandSolder, symbol Device:C
- removed D2: D_Schottky, Diode_SMD:D_SOD-323_HandSoldering, symbol Device:D_Schottky
- removed FB1: FerriteBead, Inductor_SMD:L_1206_3216Metric_Pad1.22x1.90mm_HandSolder, symbol Device:FerriteBead
- removed J2: USB4125-GF-A-0190_REVA2, GDH Connectors:GCT_USB4125-GF-A-0190_REVA2, symbol GDH Connectors:USB4125-GF-A-0190_REVA2
- removed R1, R2: 5.1k, Resistor_SMD:R_0805_2012Metric_Pad1.20x1.40mm_HandSolder, symbol Device:R
- U1: symbol GDH Amplifiers:ADA4857-1YRZ-R7 -> GDH Amplifiers:ADA4857
Connections:
- net VDD: no longer RA1.1
- new net V_{DD}: RA1.1
Other:
- added sheet USB-C Power (usb-c.kicad_sch)
- note removed: "USB-C Power Input (5V)"
- moved on the sheet: C1, C2, C3, C6, C_IN1, C_OUT1, C_VREF_A1, C_VREF_B1, D1, J3, RA1, RB1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
